File: Avionics/Quad Flight Computer/QuadFCv1.sch (EAGLE design)
At the start: 1 part, among them U1 LPC1769LQFP100

Commit message: Added LPC4337 to library. Damn that took a long time
Parts:
- added C1: 1uF, SparkFun-Passives:CAP0402-CAP
- added L1: 10uH, SparkFun-Passives:INDUCTOR0402
Connections:
- new net 3.3V: L1.1, U1.VBAT, U1.VDD_3V3@1, U1.VDD_3V3@2, U1.VDD_3V3@3, U1.VDD_3V3@4, U1.VDD_REG_3V3@1, U1.VDD_REG_3V3@2
- new net GND: C1.2, U1.VREFN, U1.VSS@1, U1.VSS@2, U1.VSS@3, U1.VSS@4, U1.VSS@5, U1.VSS@6, U1.VSSA
- new net N$1: C1.1, L1.2, U1.VDDA, U1.VREFP
Changed lines of the file:
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@@
 <parts>
 <part name="U1" library="Shared Libraries" deviceset="LPC1769" device="LQFP100"/>
+<part name="L1" library="SparkFun-Passives" deviceset="INDUCTOR" device="0402" value="10uH"/>
+<part name="C1" library="SparkFun-Passives" deviceset="CAP" device="0402-CAP" value="1uF"/>
+<part name="GND2" library="SparkFun-Aesthetics" deviceset="DGND" device=""/>
+<part name="SUPPLY2" library="SparkFun-Aesthetics" deviceset="3.3V" device=""/>
+<part name="GND3" library="SparkFun-Aesthetics" deviceset="DGND" device=""/>
+<part name="GND1" library="SparkFun-Aesthetics" deviceset="DGND" device=""/>
 </parts>
 <sheets>
 <sheet>
+<description>MCU
+Main flight processor with required circuitry and labeled IO</description>
 <plain>
 </plain>
 <instances>
 <instance part="U1" gate="G$1" x="0" y="0"/>
+<instance part="L1" gate="G$1" x="-73.66" y="-30.48"/>
+<instance part="C1" gate="G$1" x="-73.66" y="-48.26"/>
+<instance part="GND2" gate="G$1" x="-73.66" y="-55.88"/>
+<instance part="SUPPLY2" gate="G$1" x="-73.66" y="-20.32"/>
+<instance part="GND3" gate="G$1" x="-55.88" y="-68.58" rot="R270"/>
+<instance part="GND1" gate="G$1" x="-55.88" y="-48.26" rot="R270"/>
 </instances>
 <busses>
+</busses>
+<nets>
+<net name="GND" class="0">
+<segment>
+<pinref part="C1" gate="G$1" pin="2"/>
+<pinref part="GND2" gate="G$1" pin="GND"/>
+<wire x1="-73.66" y1="-53.34" x2="-73.66" y2="-50.8" width="0.1524" layer="91"/>
+</segment>
+<segment>
+<pinref part="GND3" gate="G$1" pin="GND"/>
+<pinref part="U1" gate="G$1" pin="VREFN"/>
+<wire x1="-53.34" y1="-68.58" x2="-45.72" y2="-68.58" width="0.1524" layer="91"/>
+</segment>
+<segment>
+<pinref part="U1" gate="G$1" pin="VSSA"/>
+<wire x1="-45.72" y1="-43.18" x2="-53.34" y2="-43.18" width="0.1524" layer="91"/>
+<wire x1="-53.34" y1="-43.18" x2="-53.34" y2="-48.26" width="0.1524" layer="91"/>
+<pinref part="U1" gate="G$1" pin="VSS@6"/>
+<wire x1="-53.34" y1="-48.26" x2="-53.34" y2="-50.8" width="0.1524" layer="91"/>
+<wire x1="-53.34" y1="-50.8" x2="-53.34" y2="-53.34" width="0.1524" layer="91"/>
+<wire x1="-53.34" y1="-53.34" x2="-53.34" y2="-55.88" width="0.1524" layer="91"/>
+<wire x1="-53.34" y1="-55.88" x2="-53.34" y2="-58.42" width="0.1524" layer="91"/>
+<wire x1="-53.34" y1="-58.42" x2="-53.34" y2="-60.96" width="0.1524" layer="91"/>
+<wire x1="-53.34" y1="-60.96" x2="-45.72" y2="-60.96" width="0.1524" layer="91"/>
+<pinref part="U1" gate="G$1" pin="VSS@5"/>
+<wire x1="-45.72" y1="-58.42" x2="-53.34" y2="-58.42" width="0.1524" layer="91"/>
+<pinref part="U1" gate="G$1" pin="VSS@4"/>
+<wire x1="-45.72" y1="-55.88" x2="-53.34" y2="-55.88" width="0.1524" layer="91"/>
+<pinref part="U1" gate="G$1" pin="VSS@3"/>
+<wire x1="-45.72" y1="-53.34" x2="-53.34" y2="-53.34" width="0.1524" layer="91"/>
+<pinref part="U1" gate="G$1" pin="VSS@2"/>
+<wire x1="-45.72" y1="-50.8" x2="-53.34" y2="-50.8" width="0.1524" layer="91"/>
+<pinref part="U1" gate="G$1" pin="VSS@1"/>
+<wire x1="-45.72" y1="-48.26" x2="-53.34" y2="-48.26" width="0.1524" layer="91"/>
+<junction x="-53.34" y="-58.42"/>
+<junction x="-53.34" y="-55.88"/>
+<junction x="-53.34" y="-53.34"/>
+<junction x="-53.34" y="-50.8"/>
+<junction x="-53.34" y="-48.26"/>
+<pinref part="GND1" gate="G$1" pin="GND"/>
+</segment>
+</net>
+<net name="N$1" class="0">
+<segment>
+<pinref part="U1" gate="G$1" pin="VDDA"/>
+<pinref part="L1" gate="G$1" pin="2"/>
+<wire x1="-45.72" y1="-40.64" x2="-73.66" y2="-40.64" width="0.1524" layer="91"/>
+<pinref part="C1" gate="G$1" pin="1"/>
+<wire x1="-73.66" y1="-40.64" x2="-73.66" y2="-38.1" width="0.1524" layer="91"/>
+<wire x1="-73.66" y1="-43.18" x2="-73.66" y2="-40.64" width="0.1524" layer="91"/>
+<junction x="-73.66" y="-40.64"/>
+<pinref part="U1" gate="G$1" pin="VREFP"/>
+<wire x1="-45.72" y1="-66.04" x2="-81.28" y2="-66.04" width="0.1524" layer="91"/>
+<wire x1="-81.28" y1="-66.04" x2="-81.28" y2="-40.64" width="0.1524" layer="91"/>
+<wire x1="-81.28" y1="-40.64" x2="-73.66" y2="-40.64" width="0.1524" layer="91"/>
+</segment>
+</net>
+<net name="3.3V" class="0">
+<segment>
+<pinref part="U1" gate="G$1" pin="VDD_3V3@1"/>
+<wire x1="-53.34" y1="-22.86" x2="-45.72" y2="-22.86" width="0.1524" layer="91"/>
+<wire x1="-53.34" y1="-22.86" x2="-53.34" y2="-25.4" width="0.1524" layer="91"/>
+<pinref part="U1" gate="G$1" pin="VDD_3V3@2"/>
+<wire x1="-53.34" y1="-25.4" x2="-45.72" y2="-25.4" width="0.1524" layer="91"/>
+<pinref part="U1" gate="G$1" pin="VDD_3V3@3"/>
+<wire x1="-45.72" y1="-27.94" x2="-53.34" y2="-27.94" width="0.1524" layer="91"/>
+<wire x1="-53.34" y1="-27.94" x2="-53.34" y2="-25.4" width="0.1524" layer="91"/>
+<pinref part="U1" gate="G$1" pin="VDD_3V3@4"/>
+<wire x1="-45.72" y1="-30.48" x2="-53.34" y2="-30.48" width="0.1524" layer="91"/>
+<wire x1="-53.34" y1="-30.48" x2="-53.34" y2="-27.94" width="0.1524" layer="91"/>
+<pinref part="U1" gate="G$1" pin="VDD_REG_3V3@1"/>
+<wire x1="-45.72" y1="-33.02" x2="-53.34" y2="-33.02" width="0.1524" layer="91"/>
+<wire x1="-53.34" y1="-33.02" x2="-53.34" y2="-30.48" width="0.1524" layer="91"/>
+<pinref part="U1" gate="G$1" pin="VDD_REG_3V3@2"/>
+<wire x1="-45.72" y1="-35.56" x2="-53.34" y2="-35.56" width="0.1524" layer="91"/>
+<wire x1="-53.34" y1="-35.56" x2="-53.34" y2="-33.02" width="0.1524" layer="91"/>
+<junction x="-53.34" y="-33.02"/>
+<junction x="-53.34" y="-30.48"/>
+<junction x="-53.34" y="-27.94"/>
+<junction x="-53.34" y="-25.4"/>
+<pinref part="L1" gate="G$1" pin="1"/>
+<wire x1="-53.34" y1="-22.86" x2="-73.66" y2="-22.86" width="0.1524" layer="91"/>
+<pinref part="SUPPLY2" gate="G$1" pin="3.3V"/>
+<wire x1="-73.66" y1="-22.86" x2="-73.66" y2="-20.32" width="0.1524" layer="91"/>
+<junction x="-73.66" y="-22.86"/>
+<junction x="-53.34" y="-22.86"/>
+<pinref part="U1" gate="G$1" pin="VBAT"/>
+<wire x1="-45.72" y1="-73.66" x2="-88.9" y2="-73.66" width="0.1524" layer="91"/>
+<wire x1="-88.9" y1="-73.66" x2="-88.9" y2="-22.86" width="0.1524" layer="91"/>
+<wire x1="-88.9" y1="-22.86" x2="-73.66" y2="-22.86" width="0.1524" layer="91"/>
+</segment>
+</net>
+</nets>
+</sheet>
+<sheet>
+<description>Power
+Regulators, isolation, and jumper options</description>
+<plain>
+</plain>
+<instances>
+</instances>
+<busses>

Commit message: Broke out all of the flight computer MCU ports and assigned the dedicated signals for use internally.
Parts:
- added C10, C15, C4, C5, C6, C7, C8, C9: 0.1uF, SparkFun-Capacitors:CAP0603-CAP
- added C11, C12: 18pF, SparkFun-Capacitors:CAP0603-CAP
- added C2: 3.3uF, SparkFun-Capacitors:CAP0603-CAP
- added C3: 1uF, SparkFun-Capacitors:CAP0603-CAP
- added JP1, JP2: M10", SparkFun-Connectors:M10"
- added R1, R2, R22: 10K, SparkFun-Resistors:RESISTOR0603-RES
- added R10, R11, R12, R14, R15, R16, R17, R18, R19, R20, R21, R5, R6, R7, R8, R9: 220, SparkFun-Resistors:RESISTOR0603-RES
- added R13, R4: 0, SparkFun-Resistors:RESISTOR0805-RES
- added R23: 49.9K, SparkFun-Resistors:RESISTOR0603-RES
- added STANDOFF1, STANDOFF2, STANDOFF3, STANDOFF4: STAND-OFF, SparkFun-Electromechanical:STAND-OFF
- added SW1: 2-1437565-9, Shared Libraries:2-1437565-9
- added U2: TM4C123GH6PZ, Shared Libraries:TM4C123GH6PZ
- added Y1: 32.768KHZ, Shared Libraries:ECS-.327-12.5-34B
- added Y2: AWSCR-20.00CW-T, Shared Libraries:AWSCR-20.00CW-T
- C1: device SparkFun-Passives:CAP0402-CAP -> SparkFun-Passives:CAP0603-CAP
- L1: device SparkFun-Passives:INDUCTOR0402 -> SparkFun-Passives:INDUCTOR0603
- U1: value LPC1769LQFP100 -> 74LVC4245APW; device Shared Libraries:LPC1769LQFP100 -> Shared Libraries:74LVC4245APW
Connections:
- new net 5V: R13.2, R4.2, U1VCC5.1
- new net FC_AIN0: U2PORTE.PE3/AIN0
- new net FC_AIN1: U2PORTE.PE2/AIN1
- new net FC_AIN20: U2PORTE.PE7/AIN20/CAN1TX/U1RI
- new net FC_AIN21: U2PORTE.PE6/AIN21/CAN1RX
- new net FC_AIN4: U2PORTD.PD7/AIN4/M0FAULT1/NMI/PHB0/U2TX/WT5CCP1
- new net FC_AIN5: U2PORTD.PD6/AIN5/M0FAULT0/PHA0/U2RX/WT5CCP0
- new net FC_I2C3SCL: U2PORTG.PG0/I2C3SCL/M1FAULT1/PHA1/T4CCP0
- new net FC_I2C3SDA: U2PORTG.PG1/I2C3SDA/M1FAULT2/PHB1/T4CCP1
- new net FC_JTAG_TCK: U2PORTC.PC0/SWCLK/T4CCP0/TCK
- new net FC_JTAG_TDI: U2PORTC.PC2/T5CCP0/TDI
- new net FC_JTAG_TDO: U2PORTC.PC3/SWO/T5CCP1/TDO
- new net FC_JTAG_TMS: U2PORTC.PC1/SWDIO/T4CCP1/TMS
- new net FC_PA6: U2PORTA.PA6/I2C1SCL/M1PWM2
- new net FC_PA7: U2PORTA.PA7/I2C1SDA/M1PWM3
- new net FC_PB2: U2PORTB.PB2/I2C0SCL/T3CCP0
- new net FC_PB3: U2PORTB.PB3/I2C0SDA/T3CCP1
- new net FC_PB4: U2PORTB.PB4/AIN10/CAN0RX/M0PWM2/SSI2CLK/T1CCP0
- new net FC_PB5: U2PORTB.PB5/AIN11/CAN0TX/M0PWM3/SSI2FSS/T1CCP1
- new net FC_PD0: U2PORTD.PD0/AIN15/I2C3SCL/M0PWM6/M1PWM0/SSI1CLK/SSI3CLK/WT2CCP0
- new net FC_PD1: U2PORTD.PD1/AIN14/I2C3SDA/M0PWM7/M1PWM1/SSI1FSS/SSI3FSS/WT2CCP1
- new net FC_PD2: U2PORTD.PD2/AIN13/M0FAULT0/SSI1RX/SSI3RX/USB0EPEN/WT3CCP0
- new net FC_PD3: U2PORTD.PD3/AIN12/IDX0/SSI1TX/SSI3TX/USB0PFLT/WT3CCP1
- new net FC_PD4: U2PORTD.PD4/AIN7/U6RX/WT4CCP0
- new net FC_PD5: U2PORTD.PD5/AIN6/U6TX/WT4CCP1
- new net FC_PE4: U2PORTE.PE4/AIN9/CAN0RX/I2C2SCL/M0PWM4/M1PWM2/U5RX
- new net FC_PE5: U2PORTE.PE5/AIN8/CAN0TX/I2C2SDA/M0PWM5/M1PWM3/U5TX
- new net FC_PF0: U2PORTF.PF0/C0O/CAN0RX/M1PWM4/NMI/PHA0/SSI1RX/T0CCP0/TRD2/U1RTS
- new net FC_PF1: U2PORTF.PF1/C1O/M1PWM5/PHB0/SSI1TX/T0CCP1/TRD1/U1CTS
- new net FC_PF2: U2PORTF.PF2/C2O/M0FAULT0/M1PWM6/SSI1CLK/T1CCP0/TRD0/U1DCD
- new net FC_PF3: U2PORTF.PF3/CAN0TX/M0FAULT1/M1PWM7/SSI1FSS/T1CCP1/TRCLK/U1DSR
- new net FC_PF4: U2PORTF.PF4/IDX0/M0FAULT2/M1FAULT0/T2CCP0/TRD3/U1DTR/USB0EPEN
- new net FC_PF5: U2PORTF.PF5/M0FAULT3/T2CCP1/USB0PFLT
- new net FC_PF6: U2PORTF.PF6/I2C2SCL/T3CCP0
- new net FC_PF7: U2PORTF.PF7/I2C2SDA/M1FAULT0/T3CCP1
- new net FC_PG2: U2PORTG.PG2/I2C4SCL/M0FAULT1/M1PWM0/T5CCP0
- new net FC_PG3: U2PORTG.PG3/I2C4SDA/M0FAULT2/M1PWM1/PHA1/T5CCP1
- new net FC_PG4: U2PORTG.PG4/I2C1SCL/M0PWM4/M1PWM2/PHB1/U2RX/USB0EPEN/MT0CCP0
- new net FC_PG5: U2PORTG.PG5/I2C1SDA/IDX1/M0PWM5/M1PWM3/U2TX/USB0PFLT/WT0CCP1
- new net FC_PG6: U2PORTG.PG6/C2+/I2C5SCL/M0PWM6/WT1CCP0
- new net FC_PG7: U2PORTG.PG7/C2-/I2C5SDA/IDX1/M0PWM7/WT1CCP1
- new net FC_PJ2: U2PORTJ.PJ2/IDX0/T2CCP0/U5RX
- new net FC_PWMOUT1: U1G$1.B1, U2PORTH.PH0/AIN16/M0FAULT0/M0PWM0/SSI3CLK/WT2CCP0
- new net FC_PWMOUT2: U1G$1.B2, U2PORTH.PH1/AIN17/IDX0/M0FAULT1/M0PWM1/SSI3FSS/WT2CCP1
- new net FC_PWMOUT3: U1G$1.B3, U2PORTH.PH2/AIN18/M0FAULT2/M0PWM2/SSI3RX/WT5CCP0
- new net FC_PWMOUT4: U1G$1.B4, U2PORTH.PH3/AIN19/M0FAULT3/M0PWM3/SSI3TX/WT5CCP1
- new net FC_PWMOUT5: U1G$1.B5, U2PORTH.PH4/M0PWM4/PHA0/SSI2CLK/WT3CCP0
- new net FC_PWMOUT6: U1G$1.B6, U2PORTH.PH5/M0PWM5/PHB0/SSI2FSS/WT3CCP1
- new net FC_PWMOUT7: U1G$1.B7, U2PORTH.PH6/M0PWM6/SSI2RX/WT4CCP0
- new net FC_PWMOUT8: U1G$1.B8, U2PORTH.PH7/M0PWM7/SSI2TX/WT4CCP1
- new net FC_PWMOUT_ARM_L: R23.1, U1G$1.OE_L
- new net FC_RESET_L: C15.1, R1.1, SW1.1, SW1.2, U2SPECIAL.RST_L
- new net FC_SSI0CLK: U2PORTA.PA2/SSI0CLK
- new net FC_SSI0FSS: U2PORTA.PA3/SSI0FSS
- new net FC_SSI0RX: U2PORTA.PA4/SSI0RX
- new net FC_SSI0TX: U2PORTA.PA5/SSI0TX
- new net FC_SSI3CLK: U2PORTK.PK0/M1FAULT0/SSI3CLK
- new net FC_SSI3FSS: U2PORTK.PK1/M1FAULT1/SSI3FSS
- new net FC_SSI3RX: U2PORTK.PK2/M1FAULT2/SSI3RX
- new net FC_SSI3TX: U2PORTK.PK3/M1FAULT3/SSI3TX
- new net FC_U0RX: U2PORTA.PA0/CAN1RX/U0RX
- new net FC_U0TX: U2PORTA.PA1/CAN1TX/U0TX
- new net FC_U1RX: U2PORTC.PC4/C1-/IDX1/M0PWM6/U1RTS/U1RX/U4RX/WT0CCP0
- new net FC_U1TX: U2PORTC.PC5/C1+/M0PWM7/PHA1/U1CTS/U1TX/U4TX/WT0CCP1
- new net FC_U3RX: U2PORTC.PC6/C0+/PHB1/U3RX/USB0EPEN/WT1CCP0
- new net FC_U3TX: U2PORTC.PC7/C0-/U3TX/USB0PFLT/WT1CCP1
- new net FC_U7RX: U2PORTE.PE0/AIN3/U7RX
- new net FC_U7TX: U2PORTE.PE1/AIN2/U7TX
- new net FC_USB0DM: U2PORTJ.PJ0/T1CCP0/U4RX/USB0DM
- new net FC_USB0DP: U2PORTJ.PJ1/T1CCP1/U4TX/USB0DP
- new net FC_USB0ID: U2PORTB.PB0/T2CCP0/U1RX/USB0ID
- new net FC_USB0VBUS: U2PORTB.PB1/T2CCP1/U1TX/USB0VBUS
- new net GNDX: C11.2, C12.2, U2PWR.GNDX
- new net N$10: JP2.4, R15.2
- new net N$11: JP2.5, R16.2
- new net N$12: JP2.6, R17.2
- new net N$13: JP2.7, R18.2
- new net N$14: JP2.8, R19.2
- new net N$15: JP2.9, R20.2
- new net N$16: JP2.10, R21.2
- new net N$17: C1.2, L1.1, U2PWR.VREFA+
- new net N$18: C2.1, U2PWR.VDDC@1, U2PWR.VDDC@2
- new net N$19: C12.1, U2SPECIAL.XOSC1, Y1.2
- new net N$2: JP1.4, R6.2
- new net N$20: R22.2, U1G$1.DIR
- new net N$21: C11.1, U2SPECIAL.XOSC0, Y1.1
- new net N$22: R2.1, U2SPECIAL.WAKE_L
- new net N$23: JP1.2, R4.1
- new net N$24: U2SPECIAL.OSC0, Y2.1
- new net N$25: U2SPECIAL.OSC1, Y2.3
- new net N$26: JP2.2, R13.1
- new net N$3: JP1.5, R7.2
- new net N$4: JP1.6, R8.2
- new net N$5: JP1.7, R9.2
- new net N$6: JP1.8, R10.2
- new net N$7: JP1.9, R11.2
- new net N$8: JP1.10, R12.2
- new net N$9: JP2.3, R14.2
- new net PWMIN1: R5.1
- new net PWMIN2: R6.1
- new net PWMIN3: R7.1
- new net PWMIN4: R8.1
- new net PWMIN5: R9.1
- new net PWMIN6: R10.1
- new net PWMIN7: R11.1
- new net PWMIN8: R12.1
- new net PWMOUT1: R14.1, U1G$1.A1
- new net PWMOUT2: R15.1, U1G$1.A2
- new net PWMOUT3: R16.1, U1G$1.A3
- new net PWMOUT4: R17.1, U1G$1.A4
- new net PWMOUT5: R18.1, U1G$1.A5
- new net PWMOUT6: R19.1, U1G$1.A6
- new net PWMOUT7: R20.1, U1G$1.A7
- new net PWMOUT8: R21.1, U1G$1.A8
- net 3.3V: now also C10.1, C3.1, C4.1, C5.1, C6.1, C7.1, C8.1, C9.1, L1.2, R1.2, R23.2, U1VCC3@1.1, U1VCC3@2.1, U2PWR.VBAT, U2PWR.VDD@1, U2PWR.VDD@2, U2PWR.VDD@3, U2PWR.VDD@4, U2PWR.VDD@5, U2PWR.VDD@6, U2PWR.VDD@7, U2PWR.VDD@8, U2PWR.VDDA; no longer L1.1, U1.VBAT, U1.VDD_3V3@1, U1.VDD_3V3@2, U1.VDD_3V3@3, U1.VDD_3V3@4, U1.VDD_REG_3V3@1, U1.VDD_REG_3V3@2
- net GND: now also C1.1, C10.2, C15.2, C2.2, C3.2, C4.2, C5.2, C6.2, C7.2, C8.2, C9.2, JP1.1, JP2.1, R2.2, R22.1, SW1.3, SW1.4, U1GND@1.1, U1GND@2.1, U1GND@3.1, U2PWR.GND@1, U2PWR.GND@2, U2PWR.GND@3, U2PWR.GND@4, U2PWR.GND@5, U2PWR.GND@6, U2PWR.GND@7, U2PWR.GND@8, U2PWR.GNDA, U2PWR.VREFA-, Y2.2; no longer C1.2, U1.VREFN, U1.VSS@1, U1.VSS@2, U1.VSS@3, U1.VSS@4, U1.VSS@5, U1.VSS@6, U1.VSSA
- net N$1: now also JP1.3, R5.2; no longer C1.1, L1.2, U1.VDDA, U1.VREFP

Commit message: Added PPM encoder framework from Ardupilot mega schematic
Parts:
- added C13: 1uF, SparkFun-Capacitors:CAP0603-CAP
- added C14, C16: .1uF, SparkFun:CAP0402-CAP
- added C17: 1uF, SparkFun:CAP0402-CAP
- added F2: 500mA, SparkFun:PTCSMD
- added J1: 10104111_MICROUSBAB, Shared Libraries:10104111_MICROUSBAB
- added LED4, LED5: ORANGE, SparkFun:LED0603
- added LED7: RED, SparkFun:LED0603
- added R24, R3: 22, Shared Libraries:RESISTOR0603-RES
- added R25, R26: 22-DNP, Shared Libraries:RESISTOR0603-RES
- added R27: 0, Shared Libraries:RESISTOR0603-RES
- added R28: 1K, SparkFun:RESISTOR0402-RES
- added R29: 1M, SparkFun:RESISTOR0402-RES
- added R30: 27, SparkFun:RESISTOR0402-RES
- added R32, R35, R46, R47, R51: 1k, SparkFun:RESISTOR0402-RES
- added R37: 10K, SparkFun:RESISTOR0402-RES
- added TP2: TPSQTP10SQ, testpad:TPSQTP10SQ
- added U10: ATMEGA32U2-MU, atmel:ATMEGA8U2-MU
- added U8: SPI_PPM, SparkFunv2:AVR_SPI_PRG_6NS
- added X3: HWB, con-molex:87758-0216
- added Y3: 16MHz, SmartPrj:RESONATORMU
- C2: value 3.3uF -> 1uF
Connections:
- new net N$27: J1.ID, R27.2
- new net N$28: J1.D-, R26.2, R3.2
- new net N$29: J1.D+, R24.2, R25.2
- new net N$30: LED5.A, R35.2
- new net N$31: LED4.A, R32.2
- new net N$32: LED7.A, R51.2
- new net PC7_LED: LED7.C, U10.(INT4/ICP1/CLK0)PC7
- new net PPM_HWB: U10.(CTS/HWB/AIN6/TO/INT7)PD7, X3-1.S
- new net PPM_OUT: R28.2, TP2.TP, U10.(OC1A/PCINT8)PC6
- new net PPM_PD0: R47.2, U10.(OC0B/INT0)PD0
- new net PPM_PD1: R46.2, U10.(AIN0/INT1)PD1
- new net PPM_RST: R37.1, U10.RESET(PC1/DW), U8.5
- new net PPM_RX: U10.(RXD1/AIN1/INT2)PD2
- new net PPM_TX: U10.(TXD1/INT3)PD3
- new net PPM_USBDM: R26.1, U10.D-
- new net PPM_USBDP: R25.1, U10.D+
- new net PPM_VBUS: U10.UVCC
- new net RXLED: LED4.C, U10.(INT5/AIN3)PD4
- new net TXLED: LED5.C, U10.(XCK/AIN4/PCINT12)PD5
- new net VUCAP: C17.1, U10.UCAP
- new net VUSB: J1.VUSB
- new net XT1: R29.2, R30.1, Y3.3
- new net XT1R: R30.2, U10.XTAL1
- new net XT2: R29.1, U10.XTAL2(PC0), Y3.1
- net 5V: now also C14.1, C16.1, R32.1, R35.1, R37.2, R51.1, U10.AVCC, U10.VCC, U8.2
- net FC_USB0DM: now also R3.1
- net FC_USB0DP: now also R24.1
- net FC_USB0ID: now also R27.1
- net GND: now also C13.2, C14.2, C16.2, C17.2, J1.GND, J1.GND@1, J1.GND@2, U10.GND, U10.PAD, U10.UGND, U8.6, X3-2.S, Y3.2
- net N$18: now also C13.1
- net PWMIN1: now also U10.(SS/PCINT0)PB0
- net PWMIN2: now also U10.(SCLK/PCINT1)PB1, U8.3
- net PWMIN3: now also U10.(PDI/MOSI/PCINT2)PB2, U8.4
- net PWMIN4: now also U10.(PD0/MISO/PCINT3)PB3, U8.1
- net PWMIN5: now also U10.(T1/PCINT4)PB4
- net PWMIN6: now also U10.(PCINT5)PB5
- net PWMIN7: now also U10.(PCINT6)PB6
- net PWMIN8: now also U10.(PCINT7/OC0A/OC1C)PB7
Other:
- note added: "Hardware Boot"

Commit message: Added IMU. Needs some work
Parts:
- added C18, C20: 0.1uF, SparkFun:CAP0402-CAP
- added C19: 2.2nF, SparkFun:CAP0402-CAP
- added C21: 10nF, SparkFun:CAP0402-CAP
- added C22: 0.22uF, SparkFun-Capacitors:CAP0603-CAP
- added C23: 4.7uF, SparkFun-Capacitors:CAP0603-CAP
- added R31: 1k, SparkFun:RESISTOR0402-RES
- added R33, R34: 10k, SparkFun:RESISTOR0402-RES
- added U3: MPU-6050-1, Testing:MPU-6050-1
- added U4: HMC5883LSMD, Shared Libraries:HMC5883LSMD
- LED5: value ORANGE -> RED
- LED7: value RED -> GREEN
- Y3: value 16MHz -> PRQC16.00SR5010X000; device SmartPrj:RESONATORMU -> Shared Libraries:PRQC16.00SR5010X000
Connections:
- removed net FC_I2C3SCL: U2PORTG.PG0/I2C3SCL/M1FAULT1/PHA1/T4CCP0
- removed net FC_I2C3SDA: U2PORTG.PG1/I2C3SDA/M1FAULT2/PHB1/T4CCP1
- new net AUX_SCL: U3.AUX_CL
- new net AUX_SDA: U3.AUX_DA
- new net FC_IMU_SCL: R33.1, U2PORTG.PG0/I2C3SCL/M1FAULT1/PHA1/T4CCP0, U3.SCL, U4.SCL
- new net FC_IMU_SDA: R34.1, U2PORTG.PG1/I2C3SDA/M1FAULT2/PHB1/T4CCP1, U3.SDA, U4.SDA
- new net FC_MAG_DRDY_L: U4.DRDY
- new net IMU_INT: U3.INT
- new net N$33: C19.1, U3.CPOUT
- new net N$34: C18.1, U3.REGOUT
- new net N$35: C23.1, U4.C1
- new net N$36: C22.1, U4.SETP
- new net N$37: C22.2, U4.SETC
- new net PPM_STATUS0: R47.1
- new net PPM_STATUS1: R46.1
- new net PPM_USB_STATUS: R31.2, U10.(AIN2/PCINT11)PC2
- new net VIO: C21.1, U3.VLOGIC
- net 3.3V: now also C20.1, R33.2, R34.2, U3.VDD, U4.S1, U4.VDD, U4.VDDIO
- net GND: now also C18.2, C19.2, C20.2, C21.2, C23.2, U3.AD0, U3.CLKIN, U3.FSYNC, U3.GND, U4.GND@1, U4.GND@2
Other:
- note added: "* Two MPU-60X0s can be connected to the same I2C bus"
- note added: "** Optional external reference clock input. Connected to GND by default."
- note added: "*** Frame synchronization digital input. Connected to GND by default"
- note added: "Alternative Address =0x69 (pin AD0 is logic high)"
- note added: "Cut trace for external clock"
- note added: "Cut trace for external sync"
- note added: "Default Address = 0x68 (pin AD0 is logic low)"
- note added: "The LSB bit of the 7 bit address is determined by the logic level on pin AD0."
