File: Avionics/Quad Power Distribution/Power Distribution.sch (EAGLE design)
At the start: 12 parts

Commit message: Added current sense circuits and most of the switching regulator.
Need to add signal splitters and output pins.
Parts:
- added BATT+, GND: 10AWG_PAD, Shared Libraries:10AWG_PAD
- added C1: 10uF, SparkFun-Capacitors:CAP0603-CAP
- added C2, C3: 22uF, SparkFun-Capacitors:CAP0603-CAP
- added C4: 0.1uF, SparkFun-Capacitors:CAP0603-CAP
- added R10, R11, R12, R9: 100K, Shared Libraries:RESISTOR0603-RES
- added R13: 124K, Shared Libraries:RESISTOR0603-RES
- added R14: 0.1, Shared Libraries:RESISTOR0603-RES
- added R15: 100k, Shared Libraries:RESISTOR0603-RES
- added R16: 56k, Shared Libraries:RESISTOR0603-RES
- added R17: 10.2k, Shared Libraries:RESISTOR0603-RES
- added R18: 52.3k, Shared Libraries:RESISTOR0603-RES
- added R19: 10k, Shared Libraries:RESISTOR0603-RES
- added R5, R6, R7, R8: 0.02 5W, Shared Libraries:RESISTORPTH-2W
- added U1, U2, U3, U4, U5: LMP8645, Shared Libraries:LMP8645
- added U6: ADP2302, Shared Libraries:ADP2302
- R1, R2, R3, R4: value 0.01 5W -> 0.02 5W
- renumbered U$1 to V1+, U$2 to V2+, U$3 to V3+, U$4 to V4+, U$5 to V1-, U$6 to V2-, U$7 to V3-, U$8 to V4-
Connections:
- new net 5V: R14.1, U1.V+, U2.V+, U3.V+, U4.V+, U5.+IN, U5.V+
- new net 5VOUT: R14.2, U5.-IN
- new net ISENSE1: U1.VOUT
- new net ISENSE2: U2.VOUT
- new net ISENSE3: U3.VOUT
- new net ISENSE4: U4.VOUT
- new net ISENSE5V: U5.VOUT
- new net N$1: R10.2, U2.RG
- new net N$10: R18.1, R19.2, U6.FB
- new net N$11: R15.1, U6.PGOOD
- new net N$12: R16.2, R17.1, U6.EN
- new net N$2: R9.2, U1.RG
- new net N$3: R11.2, U3.RG
- new net N$4: R12.2, U4.RG
- new net N$5: R13.2, U5.RG
- new net N$6: R15.2, R16.1, U6.VIN
- new net N$7: C4.1, U6.BST
- new net N$8: C4.2, U6.SW
- new net N$9: C2.1, C3.1, R18.2
- net GND: now also C2.2, C3.2, GND.P$1, R10.1, R11.1, R12.1, R13.1, R19.1, R9.1, U1.V-, U2.V-, U3.V-, U4.V-, U5.V-, U6.GND
- net V1+: now also R5.2, U1.-IN
- net V2+: now also R6.2, U2.-IN
- net V3+: now also R7.2, U3.-IN
- net V4+: now also R8.2, U4.-IN
- net VBATT+: now also BATT+.P$1, R5.1, R6.1, R7.1, R8.1, U1.+IN, U2.+IN, U3.+IN, U4.+IN
Other:
- moved on the sheet: R1, R2, R3

Commit message: Finished switcher circuit, almost there.
Parts:
- added D1: SSB43L, diode:SCHOTTKY-DIODESMD
- added L1: 10uH, SparkFun-Passives:INDUCTOR0603
- added R20, R21, R22, R23: 0, Shared Libraries:RESISTOR0603-RES
- added U10, U7, U8, U9: SERVOPLUGTHROUGHHOLE_0.1PITCH, Shared Libraries:SERVOPLUGTHROUGHHOLE_0.1PITCH
- R1, R2, R3, R4: device Shared Libraries:RESISTORPTH-5W -> Shared Libraries:RESISTORPTH-2W
Connections:
- removed net N$6: R15.2, R16.1, U6.VIN
- new net N$13: R21.2, U8.+
- new net N$14: R22.2, U9.+
- new net N$15: R23.2, U10.+
- new net S1: U7.SIG
- new net S2: U8.SIG
- new net S3: U9.SIG
- new net S4: U10.SIG
- net 5V: now also C2.1, C3.1, L1.2, R18.2
- net 5VOUT: now also R20.1, R21.1, R22.1, R23.1
- net GND: now also C1.2, D1.A, R17.2, U10.-, U7.-, U8.-, U9.-
- net N$8: now also D1.C, L1.1
- net N$9: now also R20.2, U7.+; no longer C2.1, C3.1, R18.2
- net VBATT+: now also C1.1, R15.2, R16.1, U6.VIN
Other:
- moved on the sheet: C2, C3, R18, R19

Commit message: Completed layout and routing. Adding vias later
Parts:
- added JP1: (no value), Shared Libraries:M06DF13
- added JP2: (no value), Shared Libraries:M05DF13
- R1, R2, R3, R4, R5, R6, R7, R8: device Shared Libraries:RESISTORPTH-2W -> Shared Libraries:RESISTOR2512
Connections:
- net 5VOUT: now also JP1.1
- net GND: now also JP1.2
- net ISENSE1: now also JP2.4
- net ISENSE2: now also JP2.5
- net ISENSE3: now also JP2.1
- net ISENSE4: now also JP2.2
- net ISENSE5V: now also JP2.3
- net S1: now also JP1.3
- net S2: now also JP1.4
- net S3: now also JP1.5
- net S4: now also JP1.6
Other:
- moved on the sheet: BATT+, GND, R1, R2, R20, R21, R22, R23, R3, R4, R5, R6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

Commit message: Refactored power distrib board libraries into single library
Parts:
- BATT+, GND: device Shared Libraries:10AWG_PAD -> PowerDistributionv1:10AWG_PAD
- C1, C2, C3, C4: device SparkFun-Capacitors:CAP0603-CAP -> PowerDistributionv1:CAP0603-CAP
- D1: device diode:SCHOTTKY-DIODESMD -> PowerDistributionv1:SCHOTTKY-DIODESMD
- JP1: device Shared Libraries:M06DF13 -> PowerDistributionv1:M06DF13
- JP2: device Shared Libraries:M05DF13 -> PowerDistributionv1:M05DF13
- L1: device SparkFun-Passives:INDUCTOR0603 -> PowerDistributionv1:INDUCTOR0603
- R1, R2, R3, R4, R5, R6, R7, R8: device Shared Libraries:RESISTOR2512 -> PowerDistributionv1:RESISTOR2512
- R10, R11, R12, R13, R14, R15, R16, R17, R18, R19, R20, R21, R22, R23, R9: device Shared Libraries:RESISTOR0603-RES -> PowerDistributionv1:RESISTOR0603-RES
- U1, U2, U3, U4, U5: device Shared Libraries:LMP8645 -> PowerDistributionv1:LMP8645
- U10, U7, U8, U9: device Shared Libraries:SERVOPLUGTHROUGHHOLE_0.1PITCH -> PowerDistributionv1:SERVOPLUGTHROUGHHOLE_0.1PITCH
- U6: device Shared Libraries:ADP2302 -> PowerDistributionv1:ADP2302
- V1+, V1-, V2+, V2-, V3+, V3-, V4+, V4-: device Shared Libraries:3.5MM-BULLET-PLUG5MM-PAD -> PowerDistributionv1:3.5MM-BULLET-PLUG5MM-PAD
Changed lines of the file:
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@@
 </classes>
 <parts>
-<part name="R1" library="Shared Libraries" deviceset="RESISTOR" device="2512" value="0.02 5W"/>
-<part name="R2" library="Shared Libraries" deviceset="RESISTOR" device="2512" value="0.02 5W"/>
-<part name="R3" library="Shared Libraries" deviceset="RESISTOR" device="2512" value="0.02 5W"/>
-<part name="R4" library="Shared Libraries" deviceset="RESISTOR" device="2512" value="0.02 5W"/>
-<part name="V1+" library="Shared Libraries" deviceset="3.5MM-BULLET-PLUG" device="5MM-PAD"/>
-<part name="V2+" library="Shared Libraries" deviceset="3.5MM-BULLET-PLUG" device="5MM-PAD"/>
-<part name="V3+" library="Shared Libraries" deviceset="3.5MM-BULLET-PLUG" device="5MM-PAD"/>
-<part name="V4+" library="Shared Libraries" deviceset="3.5MM-BULLET-PLUG" device="5MM-PAD"/>
-<part name="V1-" library="Shared Libraries" deviceset="3.5MM-BULLET-PLUG" device="5MM-PAD"/>
-<part name="V2-" library="Shared Libraries" deviceset="3.5MM-BULLET-PLUG" device="5MM-PAD"/>
-<part name="V3-" library="Shared Libraries" deviceset="3.5MM-BULLET-PLUG" device="5MM-PAD"/>
-<part name="V4-" library="Shared Libraries" deviceset="3.5MM-BULLET-PLUG" device="5MM-PAD"/>
-<part name="R5" library="Shared Libraries" deviceset="RESISTOR" device="2512" value="0.02 5W"/>
-<part name="R6" library="Shared Libraries" deviceset="RESISTOR" device="2512" value="0.02 5W"/>
-<part name="R7" library="Shared Libraries" deviceset="RESISTOR" device="2512" value="0.02 5W"/>
-<part name="R8" library="Shared Libraries" deviceset="RESISTOR" device="2512" value="0.02 5W"/>
-<part name="U1" library="Shared Libraries" deviceset="LMP8645" device=""/>
-<part name="R9" library="Shared Libraries" deviceset="RESISTOR" device="0603-RES" value="100K"/>
-<part name="U2" library="Shared Libraries" deviceset="LMP8645" device=""/>
-<part name="R10" library="Shared Libraries" deviceset="RESISTOR" device="0603-RES" value="100K"/>
-<part name="U3" library="Shared Libraries" deviceset="LMP8645" device=""/>
-<part name="R11" library="Shared Libraries" deviceset="RESISTOR" device="0603-RES" value="100K"/>
-<part name="U4" library="Shared Libraries" deviceset="LMP8645" device=""/>
-<part name="R12" library="Shared Libraries" deviceset="RESISTOR" device="0603-RES" value="100K"/>
-<part name="U5" library="Shared Libraries" deviceset="LMP8645" device=""/>
-<part name="R13" library="Shared Libraries" deviceset="RESISTOR" device="0603-RES" value="124K"/>
-<part name="R14" library="Shared Libraries" deviceset="RESISTOR" device="0603-RES" value="0.1"/>
-<part name="BATT+" library="Shared Libraries" deviceset="10AWG_PAD" device=""/>
-<part name="GND" library="Shared Libraries" deviceset="10AWG_PAD" device=""/>
-<part name="U6" library="Shared Libraries" deviceset="ADP2302" device=""/>
-<part name="R15" library="Shared Libraries" deviceset="RESISTOR" device="0603-RES" value="100k"/>
-<part name="R16" library="Shared Libraries" deviceset="RESISTOR" device="0603-RES" value="56k"/>
-<part name="R17" library="Shared Libraries" deviceset="RESISTOR" device="0603-RES" value="10.2k"/>
-<part name="R18" library="Shared Libraries" deviceset="RESISTOR" device="0603-RES" value="52.3k"/>
-<part name="R19" library="Shared Libraries" deviceset="RESISTOR" device="0603-RES" value="10k"/>
-<part name="C1" library="SparkFun-Capacitors" deviceset="CAP" device="0603-CAP" value="10uF"/>
-<part name="C2" library="SparkFun-Capacitors" deviceset="CAP" device="0603-CAP" value="22uF"/>
-<part name="C3" library="SparkFun-Capacitors" deviceset="CAP" device="0603-CAP" value="22uF"/>
-<part name="C4" library="SparkFun-Capacitors" deviceset="CAP" device="0603-CAP" value="0.1uF"/>
-<part name="L1" library="SparkFun-Passives" deviceset="INDUCTOR" device="0603" value="10uH"/>
-<part name="D1" library="diode" deviceset="SCHOTTKY-DIODE" device="SMD" value="SSB43L"/>
-<part name="U7" library="Shared Libraries" deviceset="SERVOPLUG" device="THROUGHHOLE_0.1PITCH"/>
-<part name="U8" library="Shared Libraries" deviceset="SERVOPLUG" device="THROUGHHOLE_0.1PITCH"/>
-<part name="U9" library="Shared Libraries" deviceset="SERVOPLUG" device="THROUGHHOLE_0.1PITCH"/>
-<part name="U10" library="Shared Libraries" deviceset="SERVOPLUG" device="THROUGHHOLE_0.1PITCH"/>
-<part name="R20" library="Shared Libraries" deviceset="RESISTOR" device="0603-RES" value="0"/>
-<part name="R21" library="Shared Libraries" deviceset="RESISTOR" device="0603-RES" value="0"/>
-<part name="R22" library="Shared Libraries" deviceset="RESISTOR" device="0603-RES" value="0"/>
-<part name="R23" library="Shared Libraries" deviceset="RESISTOR" device="0603-RES" value="0"/>
-<part name="JP1" library="Shared Libraries" deviceset="M06" device="DF13"/>
-<part name="JP2" library="Shared Libraries" deviceset="M05" device="DF13"/>
+<part name="R1" library="PowerDistributionv1" deviceset="RESISTOR" device="2512" value="0.02 5W"/>
+<part name="R2" library="PowerDistributionv1" deviceset="RESISTOR" device="2512" value="0.02 5W"/>
+<part name="R3" library="PowerDistributionv1" deviceset="RESISTOR" device="2512" value="0.02 5W"/>
+<part name="R4" library="PowerDistributionv1" deviceset="RESISTOR" device="2512" value="0.02 5W"/>
+<part name="V1+" library="PowerDistributionv1" deviceset="3.5MM-BULLET-PLUG" device="5MM-PAD"/>
+<part name="V2+" library="PowerDistributionv1" deviceset="3.5MM-BULLET-PLUG" device="5MM-PAD"/>
+<part name="V3+" library="PowerDistributionv1" deviceset="3.5MM-BULLET-PLUG" device="5MM-PAD"/>
+<part name="V4+" library="PowerDistributionv1" deviceset="3.5MM-BULLET-PLUG" device="5MM-PAD"/>
+<part name="V1-" library="PowerDistributionv1" deviceset="3.5MM-BULLET-PLUG" device="5MM-PAD"/>
+<part name="V2-" library="PowerDistributionv1" deviceset="3.5MM-BULLET-PLUG" device="5MM-PAD"/>
+<part name="V3-" library="PowerDistributionv1" deviceset="3.5MM-BULLET-PLUG" device="5MM-PAD"/>
+<part name="V4-" library="PowerDistributionv1" deviceset="3.5MM-BULLET-PLUG" device="5MM-PAD"/>
+<part name="R5" library="PowerDistributionv1" deviceset="RESISTOR" device="2512" value="0.02 5W"/>
+<part name="R6" library="PowerDistributionv1" deviceset="RESISTOR" device="2512" value="0.02 5W"/>
+<part name="R7" library="PowerDistributionv1" deviceset="RESISTOR" device="2512" value="0.02 5W"/>
+<part name="R8" library="PowerDistributionv1" deviceset="RESISTOR" device="2512" value="0.02 5W"/>
+<part name="U1" library="PowerDistributionv1" deviceset="LMP8645" device=""/>
+<part name="R9" library="PowerDistributionv1" deviceset="RESISTOR" device="0603-RES" value="100K"/>
+<part name="U2" library="PowerDistributionv1" deviceset="LMP8645" device=""/>
+<part name="R10" library="PowerDistributionv1" deviceset="RESISTOR" device="0603-RES" value="100K"/>
+<part name="U3" library="PowerDistributionv1" deviceset="LMP8645" device=""/>
+<part name="R11" library="PowerDistributionv1" deviceset="RESISTOR" device="0603-RES" value="100K"/>
+<part name="U4" library="PowerDistributionv1" deviceset="LMP8645" device=""/>
+<part name="R12" library="PowerDistributionv1" deviceset="RESISTOR" device="0603-RES" value="100K"/>
+<part name="U5" library="PowerDistributionv1" deviceset="LMP8645" device=""/>
+<part name="R13" library="PowerDistributionv1" deviceset="RESISTOR" device="0603-RES" value="124K"/>
+<part name="R14" library="PowerDistributionv1" deviceset="RESISTOR" device="0603-RES" value="0.1"/>
+<part name="BATT+" library="PowerDistributionv1" deviceset="10AWG_PAD" device=""/>
+<part name="GND" library="PowerDistributionv1" deviceset="10AWG_PAD" device=""/>
+<part name="U6" library="PowerDistributionv1" deviceset="ADP2302" device=""/>
+<part name="R15" library="PowerDistributionv1" deviceset="RESISTOR" device="0603-RES" value="100k"/>
+<part name="R16" library="PowerDistributionv1" deviceset="RESISTOR" device="0603-RES" value="56k"/>
+<part name="R17" library="PowerDistributionv1" deviceset="RESISTOR" device="0603-RES" value="10.2k"/>
+<part name="R18" library="PowerDistributionv1" deviceset="RESISTOR" device="0603-RES" value="52.3k"/>
+<part name="R19" library="PowerDistributionv1" deviceset="RESISTOR" device="0603-RES" value="10k"/>
+<part name="C1" library="PowerDistributionv1" deviceset="CAP" device="0603-CAP" value="10uF"/>
+<part name="C2" library="PowerDistributionv1" deviceset="CAP" device="0603-CAP" value="22uF"/>
+<part name="C3" library="PowerDistributionv1" deviceset="CAP" device="0603-CAP" value="22uF"/>
+<part name="C4" library="PowerDistributionv1" deviceset="CAP" device="0603-CAP" value="0.1uF"/>
+<part name="L1" library="PowerDistributionv1" deviceset="INDUCTOR" device="0603" value="10uH"/>
+<part name="D1" library="PowerDistributionv1" deviceset="SCHOTTKY-DIODE" device="SMD" value="SSB43L"/>
+<part name="U7" library="PowerDistributionv1" deviceset="SERVOPLUG" device="THROUGHHOLE_0.1PITCH"/>
+<part name="U8" library="PowerDistributionv1" deviceset="SERVOPLUG" device="THROUGHHOLE_0.1PITCH"/>
+<part name="U9" library="PowerDistributionv1" deviceset="SERVOPLUG" device="THROUGHHOLE_0.1PITCH"/>
+<part name="U10" library="PowerDistributionv1" deviceset="SERVOPLUG" device="THROUGHHOLE_0.1PITCH"/>
+<part name="R20" library="PowerDistributionv1" deviceset="RESISTOR" device="0603-RES" value="0"/>
+<part name="R21" library="PowerDistributionv1" deviceset="RESISTOR" device="0603-RES" value="0"/>
+<part name="R22" library="PowerDistributionv1" deviceset="RESISTOR" device="0603-RES" value="0"/>
+<part name="R23" library="PowerDistributionv1" deviceset="RESISTOR" device="0603-RES" value="0"/>
+<part name="JP1" library="PowerDistributionv1" deviceset="M06" device="DF13"/>
+<part name="JP2" library="PowerDistributionv1" deviceset="M05" device="DF13"/>
 </parts>
 <sheets>
