File: Avionics/Flight Computer/Power.sch (KiCad schematic (older format))
At the start: 18 parts, among them U8 TPS54232

Commit message: Finished replacement and supply tuning
Parts:
- added C96: GRM31CR61H106MA12L, Capacitors_SMD:C_1206, symbol C
Connections:
- net GND: now also C96.2
- net at C49.1, C50.1, L16.2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: now also C96.1
Other:
- moved on the sheet: C50
Changed lines of the file:
@@
 L GND #PWR0124
 U 1 1 58ABCF35
-P 4650 4150
-F 0 "#PWR0124" H 1400 -650 50  0001 C CNN
-F 1 "GND" H 4655 3977 50  0000 C CNN
-F 2 "" H 1400 -400 50  0001 C CNN
-F 3 "" H 1400 -400 50  0001 C CNN
-	1    4650 4150
+P 4900 4150
+F 0 "#PWR0124" H 1650 -650 50  0001 C CNN
+F 1 "GND" H 4905 3977 50  0000 C CNN
+F 2 "" H 1650 -400 50  0001 C CNN
+F 3 "" H 1650 -400 50  0001 C CNN
+	1    4900 4150
 	1    0    0    -1
 $EndComp
@@
 	5250 4600 5250 4750
 Wire Wire Line
-	4650 3850 4650 3750
-Connection ~ 4650 3750
+	4900 3850 4900 3750
+Connection ~ 4900 3750
 Wire Wire Line
 	3900 3850 3900 3750
@@
 U 1 1 58B727EB
 P 3900 4000
-F 0 "C49" H 4015 4099 50  0000 L CNN
-F 1 "GRM31CR61H106MA12L" V 3750 3250 50  0000 L CNN
+F 0 "C49" H 3950 4100 50  0000 L CNN
+F 1 "GRM31CR61H106MA12L" V 3750 3050 50  0000 L CNN
 F 2 "Capacitors_SMD:C_1206" H 2038 -400 50  0001 C CNN
 F 3 "" H 2000 -250 50  0001 C CNN
@@
 F 5 "20%" H 2100 -200 60  0001 L CNN "Tolerance"
 F 6 "X7R" H 2050 -100 60  0001 L CNN "Type"
-F 7 "1206" H 4015 3909 60  0000 L CNN "Package"
+F 7 "1206" H 3950 3900 60  0000 L CNN "Package"
 	1    3900 4000
 	1    0    0    -1
@@
 L C C50
 U 1 1 58B72ACD
-P 4650 4000
-F 0 "C50" H 4765 4099 50  0000 L CNN
-F 1 "UMK212BB7225KG-T" V 4500 3300 50  0000 L CNN
-F 2 "Capacitors_SMD:C_0805" H 2788 -400 50  0001 C CNN
-F 3 "" H 2750 -250 50  0001 C CNN
-F 4 "50V" H 2850 -300 60  0001 L CNN "Voltage"
-F 5 "20%" H 2850 -200 60  0001 L CNN "Tolerance"
-F 6 "X7R" H 2800 -100 60  0001 L CNN "Type"
-F 7 "0805" H 4765 3909 60  0000 L CNN "Package"
-	1    4650 4000
+P 4900 4000
+F 0 "C50" H 4950 4100 50  0000 L CNN
+F 1 "UMK212BB7225KG-T" V 4800 3150 50  0000 L CNN
+F 2 "Capacitors_SMD:C_0805" H 3038 -400 50  0001 C CNN
+F 3 "" H 3000 -250 50  0001 C CNN
+F 4 "50V" H 3100 -300 60  0001 L CNN "Voltage"
+F 5 "20%" H 3100 -200 60  0001 L CNN "Tolerance"
+F 6 "X7R" H 3050 -100 60  0001 L CNN "Type"
+F 7 "0805" H 4900 3900 60  0000 L CNN "Package"
+	1    4900 4000
 	1    0    0    -1
 $EndComp
@@
 	0    -1   -1   0
 $EndComp
+$Comp
+L C C96
+U 1 1 58E4E122
+P 4450 4000
+F 0 "C96" H 4500 4100 50  0000 L CNN
+F 1 "GRM31CR61H106MA12L" V 4300 3050 50  0000 L CNN
+F 2 "Capacitors_SMD:C_1206" H 2588 -400 50  0001 C CNN
+F 3 "" H 2550 -250 50  0001 C CNN
+F 4 "50V" H 2650 -300 60  0001 L CNN "Voltage"
+F 5 "20%" H 2650 -200 60  0001 L CNN "Tolerance"
+F 6 "X7R" H 2600 -100 60  0001 L CNN "Type"
+F 7 "1206" H 4500 3900 60  0000 L CNN "Package"
+	1    4450 4000
+	1    0    0    -1
+$EndComp
+$Comp
+L GND #PWR0138
+U 1 1 58E4E533
+P 4450 4150
+F 0 "#PWR0138" H 1200 -650 50  0001 C CNN
+F 1 "GND" H 4455 3977 50  0000 C CNN
+F 2 "" H 1200 -400 50  0001 C CNN
+F 3 "" H 1200 -400 50  0001 C CNN
+	1    4450 4150
+	1    0    0    -1
+$EndComp
+Wire Wire Line
+	4450 3850 4450 3750
+Connection ~ 4450 3750
 $EndSCHEMATC

Commit message: Minor BOM fixes.
Parts:
- U8: value TPS54232 -> TPS54232DR
Changed lines of the file:
@@
 P 6850 3900
 F 0 "U8" H 6850 4317 50  0000 C CNN
-F 1 "TPS54232" H 6850 4226 50  0000 C CNN
+F 1 "TPS54232DR" H 6850 4226 50  0000 C CNN
 F 2 "Housings_SOIC:SOIC-8_3.9x4.9mm_Pitch1.27mm" H -800 2750 50  0001 L CNN
 F 3 "http://www.ti.com/lit/ds/symlink/tps54232.pdf" H 50  2350 50  0001 C CNN
